Commit message: Add a simulation harness that measures what motions do to the pieces
Contact sensors on the arm's moving links report every touch over
gz-transport. tools/sim spawns the board and pieces (15 mm bases, 42 mm
king) from the brain's belief, runs park, a transfer or a robot reply, and
fails on any unexpected contact, any piece that should stay but moved or
tipped, and any moved piece off its believed square. It drives Gazebo
through the gz CLI, which always matches the simulator's transport version.

tools/dev/gripper_geometry.py measures the jaw opening at the grasp point
from the collision meshes; park_search.py finds park poses clear of the
board and graveyards.

Co-Authored-By: Claude Opus 5 <noreply@anthropic.com>

File: src/chessbot_description/urdf/so101_sim.urdf.xacro (robot description, xacro)
@@ -88,4 +88,35 @@
     <mu2>0.8</mu2>
   </gazebo>
+  <!--
+    Contact sensors on the moving links, for motion testing (tools/sim). Each publishes on
+    /world/<world>/model/<model>/link/<link>/sensor/<link>_contact/contact, and only
+    while the link touches something, so any message is a collision to look at,
+    except the gripper holding its target piece. The base is left out: it always
+    touches the table. Collision names follow the URDF to SDF conversion
+    (<link>_collision, <link>_collision_1, ...) of the pinned so_arm101 description.
+  -->
+  <xacro:macro name="contact_sensor" params="link count">
+    <gazebo reference="$(arg prefix)${link}">
+      <sensor name="${link}_contact" type="contact">
+        <always_on>true</always_on>
+        <update_rate>200</update_rate>
+        <contact>
+          <xacro:contact_collisions link="${link}" index="0" count="${count}" />
+        </contact>
+      </sensor>
+    </gazebo>
+  </xacro:macro>
+  <xacro:macro name="contact_collisions" params="link index count">
+    <xacro:if value="${index &lt; count}">
+      <collision>$(arg prefix)${link}_collision${'' if index == 0 else '_' + str(index)}</collision>
+      <xacro:contact_collisions link="${link}" index="${index + 1}" count="${count}" />
+    </xacro:if>
+  </xacro:macro>
+  <xacro:contact_sensor link="shoulder_link" count="3" />
+  <xacro:contact_sensor link="upper_arm_link" count="2" />
+  <xacro:contact_sensor link="lower_arm_link" count="3" />
+  <xacro:contact_sensor link="wrist_link" count="2" />
+  <xacro:contact_sensor link="gripper_link" count="2" />
+  <xacro:contact_sensor link="jaw_link" count="1" />
   <gazebo>
     <plugin filename="libgz_ros2_control-system.so" name="gz_ros2_control::GazeboSimROS2ControlPlugin">
