Commit message: Add Gemma reasoning and the real-robot stack
Reasoning: chessbot_inference serves a new Reason service from Gemma 4 E4B
(Apache-2.0) in llama-server, set up as its own pixi environment with the
CUDA build (pixi run -e llm llm). The brain adds a model-generated comment
after each of its moves, in the background, and asks Gemma to pick among
candidate moves when the camera reading is ambiguous, before asking the
player to type the move.

Real robot: the robot description is shared by sim and real, with the
Gazebo parts conditional and Feetech servo IDs for real hardware.
app.launch.xml holds the application; sim.launch.xml and the new
real.launch.xml bring up the robot underneath it, the real one with
ros2_control over feetech_ros2_driver (now in chessbot.repos) and usb_cam
components in the io container. udev rules, servo calibration and camera
settings are provided as examples; docs/hardware.md walks through setup.

Verified on the desktop: the workspace builds clean (16 packages), the real
stack runs end to end with hardware:=mock (new game, arm parked), and
reasoning is reachable in sim. Not yet re-verified: commentary text after
turning off Gemma's thinking (it came back empty before).

Also links perception with --as-needed, since the upgraded toolchain rejects
the Python binding libraries ROS message packages export, and pins
rerun_ros_bridge with the same fix.

Co-Authored-By: Claude Opus 5 <noreply@anthropic.com>

File: src/chessbot_description/urdf/so101.ros2_control.xacro (robot description, xacro)
@@ -7,5 +7,5 @@
 -->
 <robot xmlns:xacro="http://www.ros.org/wiki/xacro">
-  <xacro:macro name="chessbot_ros2_control" params="prefix hardware usb_port:='/dev/so101'">
+  <xacro:macro name="chessbot_ros2_control" params="prefix hardware usb_port:='/dev/so101' joint_config_file:=''">
     <ros2_control name="SO_ARM101" type="system">
       <hardware>
@@ -19,10 +19,13 @@
           <plugin>feetech_ros2_driver/FeetechHardwareInterface</plugin>
           <param name="usb_port">${usb_port}</param>
+          <param name="joint_config_file">${joint_config_file}</param>
         </xacro:if>
       </hardware>
-      <!-- PID gains are read by gz_ros2_control only. -->
-      <xacro:macro name="arm_joint" params="name initial_position:=0.0">
+      <!-- id and p_coefficient configure the Feetech servos; PID gains are read by gz_ros2_control only. -->
+      <xacro:macro name="arm_joint" params="name id p_coefficient:=16 initial_position:=0.0">
         <joint name="${name}">
           <param name="initial_position">${initial_position}</param>
+          <param name="id">${id}</param>
+          <param name="p_coefficient">${p_coefficient}</param>
           <command_interface name="position">
             <param name="p">100.0</param>
@@ -34,10 +37,10 @@
         </joint>
       </xacro:macro>
-      <xacro:arm_joint name="${prefix}shoulder_pan_joint" />
-      <xacro:arm_joint name="${prefix}shoulder_lift_joint" />
-      <xacro:arm_joint name="${prefix}elbow_flex_joint" />
-      <xacro:arm_joint name="${prefix}wrist_flex_joint" />
-      <xacro:arm_joint name="${prefix}wrist_roll_joint" />
-      <xacro:arm_joint name="${prefix}gripper_joint" />
+      <xacro:arm_joint name="${prefix}shoulder_pan_joint" id="1" p_coefficient="8" />
+      <xacro:arm_joint name="${prefix}shoulder_lift_joint" id="2" />
+      <xacro:arm_joint name="${prefix}elbow_flex_joint" id="3" />
+      <xacro:arm_joint name="${prefix}wrist_flex_joint" id="4" />
+      <xacro:arm_joint name="${prefix}wrist_roll_joint" id="5" />
+      <xacro:arm_joint name="${prefix}gripper_joint" id="6" />
     </ros2_control>
   </xacro:macro>

File: src/chessbot_description/urdf/so101.urdf.xacro (robot description, xacro)
@@ -1,7 +1,9 @@
 <?xml version="1.0" ?>
 <!--
-  SO-101 for chessbot, in simulation.
-  Reuses the upstream so_arm101_description macro, adds the chessbot cameras,
-  the Gazebo camera sensors, and the gz_ros2_control plugin.
+  SO-101 for chessbot, in simulation (hardware:=gazebo) or for real (hardware:=real,
+  or mock for a dry run without the arm).
+  Reuses the upstream so_arm101_description macro, adds the chessbot cameras and the
+  ros2_control description. With Gazebo it also adds the simulated camera and contact
+  sensors and the gz_ros2_control plugin.
   Adapted from ros-physical-ai/demos pai_bringup/urdf/so_arm_gz.urdf.xacro (Apache-2.0).
 -->
@@ -13,4 +15,6 @@
   <xacro:arg name="usb_port" default="/dev/so101" />
   <xacro:arg name="controllers_file" default="" />
+  <!-- Real hardware: servo calibration (homing offsets, ranges); see config/hardware. -->
+  <xacro:arg name="joint_config_file" default="" />
   <xacro:arg name="color" default="0.2 0.7 0.85 1.0" />
   <xacro:arg name="overhead_xyz" default="0.234 0.0 0.51" />
@@ -26,5 +30,7 @@
                           overhead_rpy="$(arg overhead_rpy)"
                           include_inertia="true" />
-  <xacro:chessbot_ros2_control prefix="$(arg prefix)" hardware="$(arg hardware)" usb_port="$(arg usb_port)" />
+  <xacro:chessbot_ros2_control prefix="$(arg prefix)" hardware="$(arg hardware)" usb_port="$(arg usb_port)"
+                               joint_config_file="$(arg joint_config_file)" />
+  <xacro:if value="${'$(arg hardware)' == 'gazebo'}">
   <!-- Fixed camera joints would otherwise be collapsed by the URDF to SDF conversion. -->
   <gazebo reference="overhead_camera_joint">
@@ -131,3 +137,4 @@
     </plugin>
   </gazebo>
+  </xacro:if>
 </robot>
