Commit message: Put the measured camera pose into TF
The guided workflow measured where the camera actually hangs and wrote it to the
profile, where nothing read it back: profile.py called it "the record of what was
measured, what to put in the launch". There was no transform broadcaster in the
tree at all, so perception went on using the pose the description assumed. On
this rig those two are about 200 px apart at the board - four and a half squares
- so perception was sampling one square while looking at another.

On real hardware the description now publishes the mast as overhead_camera_mount
and the calibration node broadcasts overhead_camera_link against it, from the
stored profile: once the mount appears in TF, and again whenever a calibration is
stored. In simulation the description keeps owning overhead_camera_link, because
there it is the truth rather than a guess.

Verified on the rig: base_link -> overhead_camera_link resolves to
(-0.002, -0.097, 0.329), which is the measured camera. A nominal profile comes
out as exactly identity, and the pose round trip and quaternion extraction agree
to 1e-16 over five hundred random poses.

Co-Authored-By: Claude Opus 5 <noreply@anthropic.com>

File: src/chessbot_description/urdf/cameras.xacro (robot description, xacro)
@@ -17,9 +17,15 @@
       wrist_rpy:='2.618 0.0 0.0'
       include_inertia:='false'
+      overhead_from_calibration:='false'
     ">
     <!-- Overhead camera: on the mast, looking straight down at the board centre.
          Default pose is 51 cm above the table, over the centre of a 21 cm board
          whose near edge sits 9 cm from the pan axis. -->
-    <link name="overhead_camera_link">
+    <!-- Where the mast is said to put the camera. With overhead_from_calibration, this is
+         only the mount: the calibration node publishes overhead_camera_link against it from
+         what was measured, so a camera that does not hang where this says still lands right. -->
+    <xacro:property name="overhead_child"
+                    value="${'overhead_camera_mount' if overhead_from_calibration else 'overhead_camera_link'}" />
+    <link name="${overhead_child}">
       <xacro:if value="${include_inertia}">
         <inertial>
@@ -31,5 +37,5 @@
     <joint name="overhead_camera_joint" type="fixed">
       <parent link="${prefix}base_link" />
-      <child link="overhead_camera_link" />
+      <child link="${overhead_child}" />
       <origin xyz="${overhead_xyz}" rpy="${overhead_rpy}" />
     </joint>

File: src/chessbot_description/urdf/so101.urdf.xacro (robot description, xacro)
@@ -30,5 +30,6 @@
                           overhead_xyz="$(arg overhead_xyz)"
                           overhead_rpy="$(arg overhead_rpy)"
-                          include_inertia="true" />
+                          include_inertia="true"
+                          overhead_from_calibration="${'$(arg hardware)' != 'gazebo'}" />
   <xacro:chessbot_ros2_control prefix="$(arg prefix)" hardware="$(arg hardware)" usb_port="$(arg usb_port)"
                                joint_config_file="$(arg joint_config_file)" />
