Commit message: Say which problem perception has, and give the jaw tips a frame
Asked for the board with no game started, perception answered "the board isn't
located, or hasn't been seen in a known position yet" - one message for two
unrelated problems. On the rig all sixty-four squares came back unknown while
every one of them projected inside the image, which is the second problem and
reads like the first. RESULT_NOT_LEARNED separates them, and the node says which
one it is rather than leaving it to be worked out.

The jaw tips are a frame now. gripper_frame_link is the grasp point between the
jaws and the right target for IK; the tips reach 6.3 mm past it and are what
touches a board corner, which touch-off was compensating for with a constant of
its own. gripper_tip_link carries that offset in the description instead, so it
shows up in RViz, touch_point is a transform lookup rather than arithmetic, and
gripper_tip_offset can be measured again on a rig that differs without touching
any code.

Co-Authored-By: Claude Opus 5 <noreply@anthropic.com>

File: src/chessbot_description/urdf/so101.urdf.xacro (robot description, xacro)
@@ -21,4 +21,5 @@
   <xacro:arg name="overhead_xyz" default="0.234 0.0 0.51" />
   <xacro:arg name="overhead_rpy" default="3.14159 0.0 -1.5708" />
+  <xacro:arg name="gripper_tip_offset" default="0.0063" />
   <xacro:include filename="$(find so_arm101_description)/urdf/so_arm101_macro.xacro" />
   <xacro:include filename="$(find chessbot_description)/urdf/cameras.xacro" />
@@ -27,4 +28,13 @@
   <xacro:so_arm101 prefix="$(arg prefix)" parent="world" color="$(arg color)"
                    x="0" y="0" z="0" roll="0" pitch="0" yaw="0" />
+  <!-- The IK works to gripper_frame_link, the grasp point between the jaws. The closed jaw
+       tips reach past it by this much along the approach axis (measured off the collision
+       meshes by tools/dev/gripper_geometry.py), and the tips are what touches a board corner. -->
+  <link name="$(arg prefix)gripper_tip_link" />
+  <joint name="$(arg prefix)gripper_tip_joint" type="fixed">
+    <parent link="$(arg prefix)gripper_frame_link" />
+    <child link="$(arg prefix)gripper_tip_link" />
+    <origin xyz="0 0 $(arg gripper_tip_offset)" rpy="0 0 0" />
+  </joint>
   <xacro:chessbot_cameras prefix="$(arg prefix)"
                           overhead_xyz="$(arg overhead_xyz)"
